File: POEPhone.kicad_sch (KiCad schematic)
At the start: 0 parts

Commit message: Rough initial layout
Parts:
- added J1: I2C, symbol Connector_Generic:Conn_01x04
- added R1: 100k, Resistor_THT:R_Axial_DIN0207_L6.3mm_D2.5mm_P7.62mm_Horizontal, symbol Device:R
- added U1: ~, molex-poe:molex-poe, symbol molex-poe:molex-poe
- added U2: mems-mic, mems-mic:mems-mic-round, symbol mems-mic:mems-mic
- added U3: adafruit-MAX98357, adafruit-MAX98357:adafruit-MAX98357, symbol adafruit-MAX98357:adafruit-MAX98357
Connections:
- new net: R1.1, U3.4 (GAIN)
- new net +3V3: J1.2 (Pin_2), U1.2 (3V3), U2.1 (3V), U3.1 (Vin)
- new net +5V: U1.1 (5V)
- new net GND: J1.1 (Pin_1), U1.3 (GND), U2.2 (GND), U2.6 (SEL), U3.2 (GND)
- new net I2C_SCL: J1.4 (Pin_4), U1.17 (SCL/IO16)
- new net I2C_SDA: J1.3 (Pin_3), U1.20 (SDA/IO13)
- new net I2S_AMP_DATA: U3.5 (DIN)
- new net I2S_AMP_GAIN: R1.2
- new net I2S_BCLK: U2.3 (BCLK), U3.6 (BCLK)
- new net I2S_MIC_DATA: U1.12 (RX2/I36), U2.4 (DOUT)
- new net I2S_RLCLK: U2.5 (LRCLK), U3.7 (LRC)
